File: DevShield2.7.1.brd (EAGLE design)
At the start: 56 x 51.5 mm, 58 parts, among them Q1 BC846BWT1G, SW1 BC-RESET, SW2 ARD-RESET, SW3 RECLAIM, U1 LD1117S33TR, U2 74LVC241A, U3 ETRX357, U4 SN74LVC1G32, U5 ER-OLED9.1, U6 AT45DB041D, X1 ISA HEADER, X3 RASPBERRYPI-V2-HEADERS, X4 1X5

Commit message: Updated Library and pin names for Raspberry Pi
Parts:
- IGNORE: value OLED -> ER-OLED0.91-1-OUTLINE; device BERG-Eagle_Library:ER-OLED0.91-SCREEN -> BERGCloud-OSH:ER-OLED0.91-SCREEN
- Q1: device BERG-Eagle_Library:SOT323 -> BERGCloud-OSH:SOT323
- SW1, SW2: device BERG-Eagle_Library:TE_FSMSM -> BERGCloud-OSH:TE_FSMSM
- U1: device BERG-OSH:SOT223 -> BERGCloud-OSH:SOT223
- U2: device BERG-OSH:TSSOP20 -> BERGCloud-OSH:TSSOP20
- U3: device BERG-OSH:ETRX35XSMD -> BERGCloud-OSH:ETRX35XSMD
- U4: device BERG-OSH:SC70-5 -> BERGCloud-OSH:SC70-5
- U5: value ER-OLED9.1 -> (none); device BERG-Eagle_Library:FPC15WAYOLED -> BERGCloud-OSH:FPC15WAYOLED
- X1: device BERG-OSH:SHF-105-01-L-D-SM -> BERGCloud-OSH:SHF-105-01-L-D-SM
- X2: device BERG-OSH:ARDUINO_UNO_ICSP -> BERGCloud-OSH:ARDUINO_UNO_ICSP
- X3: device BERG-Eagle_Library:RASPBERRY-PI-HEADERS -> BERGCloud-OSH:13X2_2.54MM
- X4: device BERG-OSH:1X05 -> BERGCloud-OSH:1X05
Other:
- board text added: "BERGCloud Dev Shield Copyright (c) 2013 BERG Cloud Ltd. http://bergcloud.com/ Permission is hereby granted, free of charge, to any person obtaining a copy of this hardware, software, and associated documentation files (the "Product"), to deal in the Product without restriction, including without limitation the rights to use, copy, modify, merge, publish, distribute, sublicense, and/or sell copies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"
- board text removed: "BERGCloud Dev Shield Copyright (c) 2013 BERG Cloud Ltd. http://bergcloud.com/ Permission is hereby granted, free of charge, to any person obtaining a copy of this software and associated documentation files (the "Product"), to deal in the Product without restriction, including without limitation the rights to use, copy, modify, merge, publish, distribute, sublicense, and/or sell copies of the Pro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"
